File: 445_Left_Forearm/445_Left_Forearm.kicad_pcb (KiCad board)
At the start: 2 copper layers, 24.9 x 18 mm, 2 parts, among them J1 69167-107HLF, U1 LSM6DSMTR

Commit message: Layout First Draft
Parts:
- removed J1: 69167-107HLF, 69167-107HLF:AMPHENOL_69167-107HLF
- removed U1: LSM6DSMTR, LSM6DSMTR (1):PQFN50P300X250X86-14N
- added C1: 100nF, CL21F104ZAANNNC:CAPC2012X135N, F.Cu at (148.6, 94.6)
- added C2: 100nF, CL21F104ZAANNNC:CAPC2012X135N, F.Cu at (148.6, 97.9)
- added H1: MountingHole, MountingHole:MountingHole_2mm, F.Cu at (137.8, 75.4)
- added H2: MountingHole, MountingHole:MountingHole_2mm, F.Cu at (157.6, 75.4)
- added H3: MountingHole, MountingHole:MountingHole_2mm, F.Cu at (137.8, 99.3)
- added H4: MountingHole, MountingHole:MountingHole_2mm, F.Cu at (157.6, 99.3)
- added J6: 69167-107HLF, 69167-107HLF:AMPHENOL_69167-107HLF, F.Cu at (148.8, 83.6)
- added U5: LSM6DSMTR, LSM6DSMTR (1):PQFN50P300X250X86-14N, F.Cu at (148.5, 90.2)
Routing:
- net /CS2: track 11.3 -> 0.00 mm
- net /SENSOR_3: track 0.00 -> 9.93 mm
- net /CLK: track 9.42 -> 0.00 mm
- net /INT1_3: track 0.00 -> 8.48 mm, vias 0 -> 1
- net +3.3V: track 11.0 -> 19.4 mm
- net /CLK3: track 0.00 -> 8.08 mm
- net /MOSI: track 7.79 -> 0.00 mm
- net /MOSI_3: track 0.00 -> 7.23 mm
- net /MISO_3: track 0.00 -> 6.62 mm
- net /MISO: track 5.82 -> 0.00 mm
- net GND: track 10.5 -> 11.5 mm
Other:
- board size 24.9 x 18 mm -> 24.9 x 29 mm
- board text added: "Left Forearm Version 1"

Commit message: Edits 3/12
Parts:
- moved C1 6.15 mm to (153.4, 90.8)
- moved C2 3.45 mm to (149.0, 94.5)
Routing:
- net +3.3V: track 19.4 -> 21.7 mm
- added copper zone on B.Cu, net GND
Changed lines of the file:
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@@
   (net 10 "unconnected-(U5-SDO_AUX-Pad11)")
   (footprint "CL21F104ZAANNNC:CAPC2012X135N" (layer "F.Cu")
-    (at 148.59 97.917 180)
+    (at 148.971 94.488 180)
     (property "Sheetfile" "445_Left_Forearm.kicad_sch")
     (property "Sheetname" "")
@@
   )
   (footprint "CL21F104ZAANNNC:CAPC2012X135N" (layer "F.Cu")
-    (at 148.59 94.615)
+    (at 153.416 90.805)
     (property "Sheetfile" "445_Left_Forearm.kicad_sch")
     (property "Sheetname" "")
@@
     (effects (font (size 1 1) (thickness 0.15)) (justify left bottom))
   )
+  (segment (start 147.963 91.694) (end 147.974 91.705) (width 0.25) (layer "F.Cu") (net 1))
+  (segment (start 149.623 90.92) (end 152.411 90.92) (width 0.25) (layer "F.Cu") (net 1))
+  (segment (start 149.623 91.545) (end 149.623 90.92) (width 0.25) (layer "F.Cu") (net 1))
+  (segment (start 147.81875 91.55775) (end 148.0235 91.353) (width 0.25) (layer "F.Cu") (net 1))
   (segment (start 141.224 87.376) (end 145.626 91.778) (width 0.25) (layer "F.Cu") (net 1))
-  (segment (start 148.0235 94.1) (end 147.6335 94.49) (width 0.25) (layer "F.Cu") (net 1))
-  (segment (start 147.6335 97.917) (end 147.6335 94.74) (width 0.25) (layer "F.Cu") (net 1))
+  (segment (start 149.463 91.705) (end 149.623 91.545) (width 0.25) (layer "F.Cu") (net 1))
+  (segment (start 147.963 91.08) (end 147.963 91.694) (width 0.25) (layer "F.Cu") (net 1))
+  (segment (start 152.411 90.92) (end 152.526 90.805) (width 0.25) (layer "F.Cu") (net 1))
   (segment (start 148.0235 91.353) (end 148.0235 91.228) (width 0.25) (layer "F.Cu") (net 1))
-  (segment (start 147.5985 91.778) (end 148.0235 91.353) (width 0.25) (layer "F.Cu") (net 1))
-  (segment (start 148.0235 91.207) (end 148.0235 94.1) (width 0.25) (layer "F.Cu") (net 1))
+  (segment (start 147.5985 91.778) (end 147.81875 91.55775) (width 0.25) (layer "F.Cu") (net 1))
+  (segment (start 147.974 91.705) (end 149.463 91.705) (width 0.25) (layer "F.Cu") (net 1))
+  (segment (start 148.081 91.82) (end 148.081 94.488) (width 0.25) (layer "F.Cu") (net 1))
   (segment (start 141.224 83.566) (end 141.224 87.376) (width 0.25) (layer "F.Cu") (net 1))
   (segment (start 145.626 91.778) (end 147.5985 91.778) (width 0.25) (layer "F.Cu") (net 1))
+  (segment (start 147.81875 91.55775) (end 148.081 91.82) (width 0.25) (layer "F.Cu") (net 1))
   (segment (start 146.7385 90.068) (end 147.3635 90.068) (width 0.25) (layer "F.Cu") (net 2))
   (segment (start 149.0235 90.8575) (end 149.0235 91.228) (width 0.25) (layer "F.Cu") (net 2))
@@
       )
     )
+  )
+  (zone (net 2) (net_name "GND") (layer "B.Cu") (hatch edge 0.5)
+    (priority 1)
+    (connect_pads (clearance 0.5))
+    (min_thickness 0.25) (filled_areas_thickness no)
+    (fill yes (thermal_gap 0.5) (thermal_bridge_width 0.5))
+    (polygon
+      (pts
+        (xy 137.541 77.47)
+        (xy 158.369 77.343)
+        (xy 158.369 100.457)
+        (xy 137.033 100.457)
+        (xy 137.414 77.47)
+        (xy 137.668 77.47)
+      )
+    )
