File: 445_Left_Shoulder/445_Left_Shoulder.kicad_pcb (KiCad board)
At the start: 2 copper layers, 24.9 x 18 mm, 2 parts, among them J1 69167-107HLF, U1 LSM6DSMTR

Commit message: Layout First Draft
Parts:
- removed J1: 69167-107HLF, 69167-107HLF:AMPHENOL_69167-107HLF
- removed U1: LSM6DSMTR, LSM6DSMTR (1):PQFN50P300X250X86-14N
- added C1: 100nF, CL21F104ZAANNNC:CAPC2012X135N, F.Cu at (143.8, 97.0)
- added C2: 100nF, CL21F104ZAANNNC:CAPC2012X135N, F.Cu at (143.8, 100.3)
- added H1: MountingHole, MountingHole:MountingHole_2mm, F.Cu at (133.0, 77.9)
- added H2: MountingHole, MountingHole:MountingHole_2mm, F.Cu at (152.8, 77.9)
- added H3: MountingHole, MountingHole:MountingHole_2mm, F.Cu at (133.0, 101.7)
- added H4: MountingHole, MountingHole:MountingHole_2mm, F.Cu at (152.8, 101.7)
- added J2: 69167-107HLF, 69167-107HLF:AMPHENOL_69167-107HLF, F.Cu at (144.0, 86.0)
- added U3: LSM6DSMTR, LSM6DSMTR (1):PQFN50P300X250X86-14N, F.Cu at (143.7, 92.7)
Routing:
- net /CS0: track 10.5 -> 0.00 mm
- net /SENSOR_1: track 0.00 -> 9.93 mm
- net /CLK: track 8.71 -> 0.00 mm
- net +3.3V: track 10.7 -> 19.4 mm
- net /INT1_1: track 0.00 -> 8.48 mm, vias 0 -> 1
- net /CLK1: track 0.00 -> 8.08 mm
- net /MOSI_1: track 0.00 -> 7.23 mm
- net /MOSI: track 7.08 -> 0.00 mm
- net /MISO_1: track 0.00 -> 6.62 mm
- net /MISO: track 5.52 -> 0.00 mm
- net GND: track 10.8 -> 11.5 mm
Other:
- board size 24.9 x 18 mm -> 24.9 x 29 mm
- board text added: "Left Shoulder Version 1"

Commit message: Edits 3/12
Parts:
- moved C1 6.23 mm to (149.0, 93.6)
- moved C2 3.45 mm to (144.1, 96.9)
Routing:
- net +3.3V: track 19.4 -> 22.3 mm
- added copper zone on B.Cu, net GND
Changed lines of the file:
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@@
   )
   (footprint "CL21F104ZAANNNC:CAPC2012X135N" (layer "F.Cu")
-    (at 143.764 97.028)
+    (at 148.971 93.599)
     (property "Sheetfile" "445_Left_Shoulder.kicad_sch")
     (property "Sheetname" "")
@@
   )
   (footprint "CL21F104ZAANNNC:CAPC2012X135N" (layer "F.Cu")
-    (at 143.764 100.33 180)
+    (at 144.145 96.901 180)
     (property "Sheetfile" "445_Left_Shoulder.kicad_sch")
     (property "Sheetname" "")
@@
     (effects (font (size 1 1) (thickness 0.15)) (justify left bottom))
   )
-  (segment (start 142.8075 100.33) (end 142.8075 97.153) (width 0.25) (layer "F.Cu") (net 1))
+  (segment (start 144.8575 94.106) (end 144.8575 93.481) (width 0.25) (layer "F.Cu") (net 1))
   (segment (start 136.398 85.979) (end 136.398 89.789) (width 0.25) (layer "F.Cu") (net 1))
-  (segment (start 143.1975 93.62) (end 143.1975 96.513) (width 0.25) (layer "F.Cu") (net 1))
+  (segment (start 143.1975 94.266) (end 143.2925 94.361) (width 0.25) (layer "F.Cu") (net 1))
+  (segment (start 143.1975 93.641) (end 143.1975 96.8435) (width 0.25) (layer "F.Cu") (net 1))
+  (segment (start 147.963 93.481) (end 148.081 93.599) (width 0.25) (layer "F.Cu") (net 1))
   (segment (start 140.8 94.191) (end 142.7725 94.191) (width 0.25) (layer "F.Cu") (net 1))
+  (segment (start 143.1975 93.641) (end 143.1975 94.266) (width 0.25) (layer "F.Cu") (net 1))
+  (segment (start 144.6025 94.361) (end 144.8575 94.106) (width 0.25) (layer "F.Cu") (net 1))
   (segment (start 136.398 89.789) (end 140.8 94.191) (width 0.25) (layer "F.Cu") (net 1))
-  (segment (start 143.1975 96.513) (end 142.8075 96.903) (width 0.25) (layer "F.Cu") (net 1))
+  (segment (start 144.8575 93.481) (end 147.963 93.481) (width 0.25) (layer "F.Cu") (net 1))
   (segment (start 142.7725 94.191) (end 143.1975 93.766) (width 0.25) (layer "F.Cu") (net 1))
+  (segment (start 143.2925 94.361) (end 144.6025 94.361) (width 0.25) (layer "F.Cu") (net 1))
   (segment (start 143.1975 93.766) (end 143.1975 93.641) (width 0.25) (layer "F.Cu") (net 1))
+  (segment (start 143.1975 96.8435) (end 143.255 96.901) (width 0.25) (layer "F.Cu") (net 1))
   (segment (start 144.1975 93.2705) (end 144.1975 93.641) (width 0.25) (layer "F.Cu") (net 2))
   (segment (start 142.5375 92.481) (end 142.5375 92.981) (width 0.25) (layer "F.Cu") (net 2))
@@
       )
     )
+  )
+  (zone (net 2) (net_name "GND") (layer "B.Cu") (hatch edge 0.5)
+    (priority 1)
+    (connect_pads (clearance 0.5))
+    (min_thickness 0.25) (filled_areas_thickness no)
+    (fill yes (thermal_gap 0.5) (thermal_bridge_width 0.5))
+    (polygon
+      (pts
+        (xy 132.715 80.01)
+        (xy 153.67 79.883)
+        (xy 153.67 102.616)
+        (xy 132.334 102.489)
+      )
+    )
