File: 445_Right_Forearm/445_Right_Forearm.kicad_pcb (KiCad board)
At the start: 2 copper layers, 24.9 x 18 mm, 2 parts, among them J1 69167-107HLF, U1 LSM6DSMTR

Commit message: Layout First Draft
Parts:
- removed J1: 69167-107HLF, 69167-107HLF:AMPHENOL_69167-107HLF
- removed U1: LSM6DSMTR, LSM6DSMTR (1):PQFN50P300X250X86-14N
- added C1: 100nF, CL21F104ZAANNNC:CAPC2012X135N, F.Cu at (145.6, 92.8)
- added C2: 100nF, CL21F104ZAANNNC:CAPC2012X135N, F.Cu at (145.6, 96.1)
- added H1: MountingHole, MountingHole:MountingHole_2mm, F.Cu at (134.9, 73.7)
- added H2: MountingHole, MountingHole:MountingHole_2mm, F.Cu at (154.7, 73.7)
- added H3: MountingHole, MountingHole:MountingHole_2mm, F.Cu at (134.9, 97.5)
- added H4: MountingHole, MountingHole:MountingHole_2mm, F.Cu at (154.7, 97.5)
- added J7: 69167-107HLF, 69167-107HLF:AMPHENOL_69167-107HLF, F.Cu at (145.8, 81.9)
- added U8: LSM6DSMTR, LSM6DSMTR (1):PQFN50P300X250X86-14N, F.Cu at (145.6, 88.5)
Routing:
- net /CS2: track 11.3 -> 0.00 mm
- net /SENSOR_3: track 0.00 -> 9.93 mm
- net /CLK: track 9.52 -> 0.00 mm
- net /INT1_3: track 0.00 -> 8.48 mm, vias 0 -> 1
- net +3.3V: track 11.2 -> 19.4 mm
- net /CLK3: track 0.00 -> 8.08 mm
- net /MOSI: track 7.78 -> 0.00 mm
- net /MOSI_3: track 0.00 -> 7.23 mm
- net /MISO_3: track 0.00 -> 6.62 mm
- net /MISO: track 5.96 -> 0.00 mm
- net GND: track 10.6 -> 11.5 mm
Other:
- board size 24.9 x 18 mm -> 24.9 x 29 mm
- board text added: "Right Forearm Version 1"

Commit message: Edits 3/12
Parts:
- moved C1 6.05 mm to (150.5, 89.3)
- moved C2 3.17 mm to (145.6, 93.0)
Routing:
- net +3.3V: track 19.4 -> 21.4 mm
- added copper zone on B.Cu, net GND
Changed lines of the file:
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@@
   )
   (footprint "CL21F104ZAANNNC:CAPC2012X135N" (layer "F.Cu")
-    (at 145.6025 92.837)
+    (at 150.495 89.281)
     (property "Sheetfile" "445_Right_Forearm.kicad_sch")
     (property "Sheetname" "")
@@
   )
   (footprint "CL21F104ZAANNNC:CAPC2012X135N" (layer "F.Cu")
-    (at 145.6025 96.139 180)
+    (at 145.6025 92.964 180)
     (property "Sheetfile" "445_Right_Forearm.kicad_sch")
     (property "Sheetname" "")
@@
   )
   (segment (start 138.303 81.788) (end 138.303 85.598) (width 0.25) (layer "F.Cu") (net 1))
-  (segment (start 144.7125 96.139) (end 144.7125 92.962) (width 0.25) (layer "F.Cu") (net 1))
+  (segment (start 145.1025 89.789) (end 144.7125 90.179) (width 0.25) (layer "F.Cu") (net 1))
+  (segment (start 145.1025 89.979) (end 145.1775 90.054) (width 0.25) (layer "F.Cu") (net 1))
+  (segment (start 146.7625 89.9655) (end 146.7625 89.269) (width 0.25) (layer "F.Cu") (net 1))
   (segment (start 138.303 85.598) (end 142.705 90) (width 0.25) (layer "F.Cu") (net 1))
+  (segment (start 145.1025 89.429) (end 145.1025 89.789) (width 0.25) (layer "F.Cu") (net 1))
+  (segment (start 145.1775 90.054) (end 146.674 90.054) (width 0.25) (layer "F.Cu") (net 1))
+  (segment (start 145.1025 89.789) (end 145.1025 89.979) (width 0.25) (layer "F.Cu") (net 1))
   (segment (start 145.1025 89.575) (end 145.1025 89.45) (width 0.25) (layer "F.Cu") (net 1))
-  (segment (start 145.1025 92.322) (end 144.7125 92.712) (width 0.25) (layer "F.Cu") (net 1))
-  (segment (start 145.1025 89.429) (end 145.1025 92.322) (width 0.25) (layer "F.Cu") (net 1))
+  (segment (start 149.085 89.269) (end 149.097 89.281) (width 0.25) (layer "F.Cu") (net 1))
   (segment (start 144.6775 90) (end 145.1025 89.575) (width 0.25) (layer "F.Cu") (net 1))
+  (segment (start 144.7125 90.179) (end 144.7125 92.964) (width 0.25) (layer "F.Cu") (net 1))
   (segment (start 142.705 90) (end 144.6775 90) (width 0.25) (layer "F.Cu") (net 1))
+  (segment (start 146.674 90.054) (end 146.7625 89.9655) (width 0.25) (layer "F.Cu") (net 1))
+  (segment (start 146.7625 89.269) (end 149.085 89.269) (width 0.25) (layer "F.Cu") (net 1))
   (segment (start 140.843 81.788) (end 140.843 85.3155) (width 0.25) (layer "F.Cu") (net 2))
   (segment (start 140.843 85.3155) (end 143.8175 88.29) (width 0.25) (layer "F.Cu") (net 2))
@@
       )
     )
+  )
+  (zone (net 2) (net_name "GND") (layer "B.Cu") (hatch edge 0.5)
+    (priority 1)
+    (connect_pads (clearance 0.5))
+    (min_thickness 0.25) (filled_areas_thickness no)
+    (fill yes (thermal_gap 0.5) (thermal_bridge_width 0.5))
+    (polygon
+      (pts
+        (xy 134.239 98.425)
+        (xy 155.702 98.552)
+        (xy 155.575 75.565)
+        (xy 134.366 75.692)
+      )
+    )
