File: 445_Right_Shoulder/445_Right_Shoulder.kicad_pcb (KiCad board)
At the start: 2 copper layers, 24.9 x 18 mm, 2 parts, among them J1 69167-107HLF, U1 LSM6DSMTR

Commit message: Layout First Draft
Parts:
- removed J1: 69167-107HLF, 69167-107HLF:AMPHENOL_69167-107HLF
- removed U1: LSM6DSMTR, LSM6DSMTR (1):PQFN50P300X250X86-14N
- added C1: 100nF, CL21F104ZAANNNC:CAPC2012X135N, F.Cu at (143.9, 94.4)
- added C2: 100nF, CL21F104ZAANNNC:CAPC2012X135N, F.Cu at (143.9, 97.8)
- added H1: MountingHole, MountingHole:MountingHole_2mm, F.Cu at (133.1, 75.2)
- added H2: MountingHole, MountingHole:MountingHole_2mm, F.Cu at (152.9, 75.2)
- added H3: MountingHole, MountingHole:MountingHole_2mm, F.Cu at (133.1, 99.1)
- added H4: MountingHole, MountingHole:MountingHole_2mm, F.Cu at (152.9, 99.1)
- added J3: 69167-107HLF, 69167-107HLF:AMPHENOL_69167-107HLF, F.Cu at (144.0, 83.4)
- added U6: LSM6DSMTR, LSM6DSMTR (1):PQFN50P300X250X86-14N, F.Cu at (143.8, 90.0)
Routing:
- net +3.3V: track 11.3 -> 32.1 mm
- net /SENSOR_1: track 0.00 -> 19.9 mm
- net /INT1_1: track 0.00 -> 17.0 mm, vias 0 -> 2
- net /CLK1: track 0.00 -> 16.2 mm
- net /MOSI_1: track 0.00 -> 14.5 mm
- net /MISO_1: track 0.00 -> 13.2 mm
- net GND: track 11.2 -> 23.0 mm
- net /CS0: track 11.0 -> 0.00 mm
- net /CLK: track 9.40 -> 0.00 mm
- net /MOSI: track 7.77 -> 0.00 mm
- net /MISO: track 6.10 -> 0.00 mm
Other:
- board size 24.9 x 18 mm -> 24.9 x 29 mm
- board text added: "Right Shoulder Version 1"

Commit message: Edits 3/12
Parts:
- moved C1 6.13 mm to (149.0, 90.9)
- moved C2 3.45 mm to (144.3, 94.4)
Routing:
- net +3.3V: track 32.1 -> 35.0 mm
- added copper zone on B.Cu, net GND
Changed lines of the file:
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@@
   )
   (footprint "CL21F104ZAANNNC:CAPC2012X135N" (layer "F.Cu")
-    (at 143.891 97.79 180)
+    (at 144.272 94.361 180)
     (property "Sheetfile" "445_Right_Shoulder.kicad_sch")
     (property "Sheetname" "")
@@
   )
   (footprint "CL21F104ZAANNNC:CAPC2012X135N" (layer "F.Cu")
-    (at 143.891 94.361)
+    (at 148.971 90.932)
     (property "Sheetfile" "445_Right_Shoulder.kicad_sch")
     (property "Sheetname" "")
@@
   (segment (start 136.525 87.122) (end 140.927 91.524) (width 0.25) (layer "F.Cu") (net 1))
   (segment (start 142.8995 91.524) (end 143.3245 91.099) (width 0.25) (layer "F.Cu") (net 1))
+  (segment (start 147.942 90.793) (end 148.081 90.932) (width 0.25) (layer "F.Cu") (net 1))
+  (segment (start 143.382 94.361) (end 143.3245 94.3035) (width 0.25) (layer "F.Cu") (net 1))
   (segment (start 136.525 83.312) (end 136.525 87.122) (width 0.25) (layer "F.Cu") (net 1))
   (segment (start 143.3245 91.099) (end 143.3245 90.974) (width 0.25) (layer "F.Cu") (net 1))
-  (segment (start 143.3245 90.953) (end 143.3245 93.846) (width 0.25) (layer "F.Cu") (net 1))
-  (segment (start 142.9345 97.663) (end 142.9345 94.486) (width 0.25) (layer "F.Cu") (net 1))
+  (segment (start 144.9845 91.418) (end 144.9845 90.793) (width 0.25) (layer "F.Cu") (net 1))
   (segment (start 140.927 91.524) (end 142.8995 91.524) (width 0.25) (layer "F.Cu") (net 1))
+  (segment (start 143.3245 90.953) (end 143.3245 91.503) (width 0.25) (layer "F.Cu") (net 1))
+  (segment (start 143.3995 91.578) (end 144.8245 91.578) (width 0.25) (layer "F.Cu") (net 1))
   (segment (start 143.3245 91.099) (end 143.3245 90.974) (width 0.25) (layer "F.Cu") (net 1))
+  (segment (start 144.9845 90.793) (end 147.942 90.793) (width 0.25) (layer "F.Cu") (net 1))
   (segment (start 136.525 83.312) (end 136.525 87.122) (width 0.25) (layer "F.Cu") (net 1))
   (segment (start 140.927 91.524) (end 142.8995 91.524) (width 0.25) (layer "F.Cu") (net 1))
-  (segment (start 143.3245 93.846) (end 142.9345 94.236) (width 0.25) (layer "F.Cu") (net 1))
+  (segment (start 143.3245 91.503) (end 143.3995 91.578) (width 0.25) (layer "F.Cu") (net 1))
+  (segment (start 143.3245 94.3035) (end 143.3245 90.953) (width 0.25) (layer "F.Cu") (net 1))
+  (segment (start 144.8245 91.578) (end 144.9845 91.418) (width 0.25) (layer "F.Cu") (net 1))
   (segment (start 136.525 87.122) (end 140.927 91.524) (width 0.25) (layer "F.Cu") (net 1))
   (segment (start 144.035 90.314) (end 144.3245 90.6035) (width 0.25) (layer "F.Cu") (net 2))
@@
         (xy 132.715 77.216)
         (xy 153.797 77.089)
-        (xy 153.797 100.076)
-        (xy 132.461 99.949)
+        (xy 153.924 96.647)
+        (xy 132.588 96.52)
       )
     )
+  )
+  (zone (net 2) (net_name "GND") (layer "B.Cu") (hatch edge 0.5)
+    (priority 1)
+    (connect_pads (clearance 0.5))
+    (min_thickness 0.25) (filled_areas_thickness no)
+    (fill yes (thermal_gap 0.5) (thermal_bridge_width 0.5))
+    (polygon
+      (pts
+        (xy 132.715 77.216)
+        (xy 153.67 77.089)
+        (xy 154.051 96.647)
+        (xy 132.588 96.52)
+      )
+    )
