File: Forearm_Shoulder Boards/Forearm_Shoulder Boards.kicad_pcb (KiCad board)
At the start: 2 copper layers, 24.9 x 29 mm, 8 parts, among them J6 69167-107HLF, U5 LSM6DSMTR

Commit message: Version 2
Other:
- board text removed: "Left Forearm Version 1"
Changed lines of the file:
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@@
       (plot_on_all_layers_selection 0x0000000_00000000)
       (disableapertmacros false)
-      (usegerberextensions false)
-      (usegerberattributes true)
-      (usegerberadvancedattributes true)
-      (creategerberjobfile true)
+      (usegerberextensions true)
+      (usegerberattributes false)
+      (usegerberadvancedattributes false)
+      (creategerberjobfile false)
       (dashed_line_dash_ratio 12.000000)
       (dashed_line_gap_ratio 3.000000)
@@
       (psa4output false)
       (plotreference true)
-      (plotvalue true)
+      (plotvalue false)
       (plotinvisibletext false)
       (sketchpadsonfab false)
-      (subtractmaskfromsilk false)
+      (subtractmaskfromsilk true)
       (outputformat 1)
       (mirror false)
-      (drillshape 1)
+      (drillshape 0)
       (scaleselection 1)
       (outputdirectory "")
@@
     (property "ki_keywords" "capacitor cap")
     (attr smd)
-    (fp_text reference "C2" (at 0 -1.524) (layer "F.SilkS")
+    (fp_text reference "C2" (at 0 -1.524) (layer "F.SilkS") hide
         (effects (font (size 0.64 0.64) (thickness 0.15)))
     )
@@
     (property "SnapEDA_Link" "https://www.snapeda.com/parts/69167-107HLF/Amphenol+FCI/view-part/?ref=snap")
     (attr through_hole)
-    (fp_text reference "J6" (at -8.382 3.81) (layer "F.SilkS")
+    (fp_text reference "J6" (at -8.382 3.81) (layer "F.SilkS") hide
         (effects (font (size 1 1) (thickness 0.15)))
     )
@@
     (property "ki_keywords" "capacitor cap")
     (attr smd)
-    (fp_text reference "C1" (at 0 1.524) (layer "F.SilkS")
+    (fp_text reference "C1" (at 0 1.524) (layer "F.SilkS") hide
         (effects (font (size 0.64 0.64) (thickness 0.15)))
     )
@@
     (property "SnapEDA_Link" "https://www.snapeda.com/parts/LSM6DSMTR/STMicroelectronics/view-part/?ref=snap")
     (attr smd)
-    (fp_text reference "U5" (at -1.397 2.159) (layer "F.SilkS")
+    (fp_text reference "U5" (at -1.397 2.159) (layer "F.SilkS") hide
         (effects (font (size 0.48 0.48) (thickness 0.12)))
     )
@@
   (gr_line (start 160.147 99.314) (end 160.147 75.438)
     (stroke (width 0.1) (type default)) (layer "Edge.Cuts"))
-  (gr_text "Left Forearm Version 1\n" (at 139.319 79.629) (layer "F.SilkS")
-    (effects (font (size 1 1) (thickness 0.15)) (justify left bottom))
-  )
   (segment (start 147.963 91.694) (end 147.974 91.705) (width 0.25) (layer "F.Cu") (net 1))
   (segment (start 149.623 90.92) (end 152.411 90.92) (width 0.25) (layer "F.Cu") (net 1))
