File: Bicep Boards/Bicep Boards.kicad_sch (KiCad schematic)
At the start: 17 parts, among them J1 SM02B-SRSS-TB_LF__SN_, J11 69167-107HLF, J4 69167-107HLF, J9 87583-2010RPLF, U1 ESP32-S3-WROOM-1-N16R8, U11 TS3A5018D, U12 TS3A5018D, U4 LSM6DSMTR, U9 LP2950CZ-3.3_LFT3

Commit message: Version 2
Connections:
- net +3.3V: no longer J9.01 (VCC)
- net 3.7V: now also J1.2, J9.01 (VCC); no longer J1.1
- net GND: now also J1.1; no longer J1.2
Other:
- moved on the sheet: J1, J9, U9

Commit message: sensor select pin change and silk added
Connections:
- net SENSOR_SEL: now also U1.26 (IO45); no longer U1.24 (IO47)
Changed lines of the file:
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@@
   (no_connect (at 256.54 55.88))
   (no_connect (at 110.49 167.64))
+  (no_connect (at 116.84 87.63))
   (no_connect (at 86.36 49.53))
   (no_connect (at 116.84 77.47))
@@
   (no_connect (at 116.84 52.07))
   (no_connect (at 116.84 85.09))
-  (no_connect (at 116.84 82.55))
   (wire (pts (xy 46.99 137.16) (xy 50.8 137.16))
     (stroke (width 0) (type default))
@@
     (stroke (width 0) (type default))
   )
-  (wire (pts (xy 118.11 87.63) (xy 116.84 87.63))
-    (stroke (width 0) (type default))
-  )
   (wire (pts (xy 232.41 121.92) (xy 228.6 121.92))
     (stroke (width 0) (type default))
@@
   )
   (wire (pts (xy 156.21 170.18) (xy 158.75 170.18))
+    (stroke (width 0) (type default))
+  )
+  (wire (pts (xy 116.84 82.55) (xy 119.38 82.55))
     (stroke (width 0) (type default))
   )
@@
     )
   )
-  (global_label "SENSOR_SEL" (shape output) (at 118.11 87.63 0) (fields_autoplaced)
-    (effects (font (size 1.27 1.27)) (justify left))
-    (property "Intersheetrefs" "${INTERSHEET_REFS}" (at 132.9484 87.63 0)
+  (global_label "SENSOR_SEL" (shape output) (at 119.38 82.55 0) (fields_autoplaced)
+    (effects (font (size 1.27 1.27)) (justify left))
+    (property "Intersheetrefs" "${INTERSHEET_REFS}" (at 134.2184 82.55 0)
       (effects (font (size 1.27 1.27)) (justify left) hide)
     )
@@
     (pin "2")
     (instances
-      (project "445_Left_Bicep"
+      (project "Bicep Boards"
         (path "/5276b365-6d0c-4da8-be37-f3b7813500d7"
           (reference "U9") (unit 1)
@@
     (pin "2")
     (instances
-      (project "445_Left_Bicep"
+      (project "Bicep Boards"
         (path "/5276b365-6d0c-4da8-be37-f3b7813500d7"
           (reference "BZ1") (unit 1)
@@
     (pin "1")
     (instances
-      (project "445_Left_Bicep"
+      (project "Bicep Boards"
         (path "/5276b365-6d0c-4da8-be37-f3b7813500d7"
           (reference "J1") (unit 1)
@@
     (pin "1")
     (instances
-      (project "445_Left_Bicep"
+      (project "Bicep Boards"
         (path "/5276b365-6d0c-4da8-be37-f3b7813500d7"
           (reference "#PWR018") (unit 1)
@@
     )
     (instances
-      (project "445_Left_Bicep"
+      (project "Bicep Boards"
         (path "/5276b365-6d0c-4da8-be37-f3b7813500d7"
           (reference "H3") (unit 1)
@@
     (pin "11")
     (instances
-      (project "445_Left_Bicep"
+      (project "Bicep Boards"
         (path "/5276b365-6d0c-4da8-be37-f3b7813500d7"
           (reference "U4") (unit 1)
@@
     (pin "3")
     (instances
-      (project "445_Left_Bicep"
+      (project "Bicep Boards"
         (path "/5276b365-6d0c-4da8-be37-f3b7813500d7"
           (reference "U11") (unit 1)
@@
     (pin "1")
     (instances
-      (project "445_Left_Bicep"
+      (project "Bicep Boards"
         (path "/5276b365-6d0c-4da8-be37-f3b7813500d7"
           (reference "#PWR05") (unit 1)
@@
     (pin "05")
     (instances
-      (project "445_Left_Bicep"
+      (project "Bicep Boards"
         (path "/5276b365-6d0c-4da8-be37-f3b7813500d7"
           (reference "J11") (unit 1)
@@
     (pin "S1")
     (instances
-      (project "445_Left_Bicep"
+      (project "Bicep Boards"
         (path "/5276b365-6d0c-4da8-be37-f3b7813500d7"
           (reference "J9") (unit 1)
@@
     )
     (instances
-      (project "445_Left_Bicep"
+      (project "Bicep Boards"
         (path "/5276b365-6d0c-4da8-be37-f3b7813500d7"
           (reference "H4") (unit 1)
@@
     )
     (instances
-      (project "445_Left_Bicep"
+      (project "Bicep Boards"
         (path "/5276b365-6d0c-4da8-be37-f3b7813500d7"
           (reference "H2") (unit 1)
@@
     (pin "1")
     (instances
-      (project "445_Left_Bicep"
+      (project "Bicep Boards"
         (path "/5276b365-6d0c-4da8-be37-f3b7813500d7"
           (reference "#PWR016") (unit 1)
@@
     (pin "1")
     (instances
-      (project "445_Left_Bicep"
+      (project "Bicep Boards"
         (path "/5276b365-6d0c-4da8-be37-f3b7813500d7"
           (reference "#PWR024") (unit 1)
@@
     (pin "1")
     (instances
-      (project "445_Left_Bicep"
+      (project "Bicep Boards"
         (path "/5276b365-6d0c-4da8-be37-f3b7813500d7"
           (reference "#PWR04") (unit 1)
@@
     (pin "15")
     (instances
-      (project "445_Left_Bicep"
+      (project "Bicep Boards"
         (path "/5276b365-6d0c-4da8-be37-f3b7813500d7"
           (reference "U12") (unit 1)
@@
     (pin "1")
     (instances
-      (project "445_Left_Bicep"
+      (project "Bicep Boards"
         (path "/5276b365-6d0c-4da8-be37-f3b7813500d7"
           (reference "#PWR02") (unit 1)
@@
     (pin "1")
     (instances
-      (project "445_Left_Bicep"
+      (project "Bicep Boards"
         (path "/5276b365-6d0c-4da8-be37-f3b7813500d7"
           (reference "#PWR07") (unit 1)
@@
     (pin "1")
     (instances
-      (project "445_Left_Bicep"
+      (project "Bicep Boards"
         (path "/5276b365-6d0c-4da8-be37-f3b7813500d7"
           (reference "#PWR015") (unit 1)
@@
     (pin "1")
     (instances
-      (project "445_Left_Bicep"
+      (project "Bicep Boards"
         (path "/5276b365-6d0c-4da8-be37-f3b7813500d7"
           (reference "#PWR03") (unit 1)
@@
     (pin "1")
     (instances
-      (project "445_Left_Bicep"
+      (project "Bicep Boards"
         (path "/5276b365-6d0c-4da8-be37-f3b7813500d7"
           (reference "#PWR01") (unit 1)
@@
     (pin "21")
     (instances
-      (project "445_Left_Bicep"
+      (project "Bicep Boards"
         (path "/5276b365-6d0c-4da8-be37-f3b7813500d7"
           (reference "U1") (unit 1)
@@
     (pin "1")
     (instances
-      (project "445_Left_Bicep"
+      (project "Bicep Boards"
         (path "/5276b365-6d0c-4da8-be37-f3b7813500d7"
           (reference "#PWR017") (unit 1)
@@
     (pin "1")
     (instances
-      (project "445_Left_Bicep"
+      (project "Bicep Boards"
         (path "/5276b365-6d0c-4da8-be37-f3b7813500d7"
           (reference "#PWR023") (unit 1)
@@
     (pin "2")
     (instances
-      (project "445_Left_Bicep"
+      (project "Bicep Boards"
         (path "/5276b365-6d0c-4da8-be37-f3b7813500d7"
           (reference "C1") (unit 1)
@@
     (pin "1")
     (instances
-      (project "445_Left_Bicep"
+      (project "Bicep Boards"
         (path "/5276b365-6d0c-4da8-be37-f3b7813500d7"
           (reference "#PWR011") (unit 1)
@@
     (pin "2")
     (instances
-      (project "445_Left_Bicep"
+      (project "Bicep Boards"
         (path "/5276b365-6d0c-4da8-be37-f3b7813500d7"
           (reference "C2") (unit 1)
@@
     (pin "1")
     (instances
-      (project "445_Left_Bicep"
+      (project "Bicep Boards"
         (path "/5276b365-6d0c-4da8-be37-f3b7813500d7"
           (reference "R1") (unit 1)
@@
     )
     (instances
-      (project "445_Left_Bicep"
+      (project "Bicep Boards"
         (path "/5276b365-6d0c-4da8-be37-f3b7813500d7"
           (reference "H1") (unit 1)
@@
     (pin "1")
     (instances
-      (project "445_Left_Bicep"
+      (project "Bicep Boards"
         (path "/5276b365-6d0c-4da8-be37-f3b7813500d7"
           (reference "#PWR010") (unit 1)
@@
     (pin "1")
     (instances
-      (project "445_Left_Bicep"
+      (project "Bicep Boards"
         (path "/5276b365-6d0c-4da8-be37-f3b7813500d7"
           (reference "#PWR014") (unit 1)
@@
     (pin "1")
     (instances
-      (project "445_Left_Bicep"
+      (project "Bicep Boards"
         (path "/5276b365-6d0c-4da8-be37-f3b7813500d7"
           (reference "#PWR06") (unit 1)
@@
     (pin "1")
     (instances
-      (project "445_Left_Bicep"
+      (project "Bicep Boards"
         (path "/5276b365-6d0c-4da8-be37-f3b7813500d7"
           (reference "#PWR020") (unit 1)
@@
     (pin "1")
     (instances
-      (project "445_Left_Bicep"
+      (project "Bicep Boards"
         (path "/5276b365-6d0c-4da8-be37-f3b7813500d7"
           (reference "#PWR021") (unit 1)
@@
     (pin "1")
     (instances
-      (project "445_Left_Bicep"
+      (project "Bicep Boards"
         (path "/5276b365-6d0c-4da8-be37-f3b7813500d7"
           (reference "#PWR08") (unit 1)
@@
     (pin "1")
     (instances
-      (project "445_Left_Bicep"
+      (project "Bicep Boards"
         (path "/5276b365-6d0c-4da8-be37-f3b7813500d7"
           (reference "#PWR09") (unit 1)
@@
     (pin "1")
     (instances
-      (project "445_Left_Bicep"
+      (project "Bicep Boards"
         (path "/5276b365-6d0c-4da8-be37-f3b7813500d7"
           (reference "#PWR022") (unit 1)
@@
     (pin "1")
     (instances
-      (project "445_Left_Bicep"
+      (project "Bicep Boards"
         (path "/5276b365-6d0c-4da8-be37-f3b7813500d7"
           (reference "#PWR012") (unit 1)
@@
     (pin "07")
     (instances
-      (project "445_Left_Bicep"
+      (project "Bicep Boards"
         (path "/5276b365-6d0c-4da8-be37-f3b7813500d7"
           (reference "J4") (unit 1)
@@
     (pin "1")
     (instances
-      (project "445_Left_Bicep"
+      (project "Bicep Boards"
         (path "/5276b365-6d0c-4da8-be37-f3b7813500d7"
           (reference "#PWR013") (unit 1)
